File: guvb-s11sd/guvb-s11sd.kicad_pcb (KiCad board)
At the start: 2 copper layers, 17.8 x 43.2 mm, 16 parts, among them P1 Digital, P2 Analog, P3 CONN_01X01, P4 CONN_01X01, P5 CONN_01X01, P6 CONN_01X01, U1 LMC6081IM, U2 LM4040

Commit message: Added turtle graphics.
Parts:
- added G***: LOGO, graphics:turtle, F.Cu at (147.0, 93.0)
